Commit message: add joint, cartesian, and force control spaces; add cartesian action features

File: assets/ur_urdf/dual_ur5e.urdf (robot description, URDF)
Before this commit: robot dual_ur5e_robot, 23 links, 22 joints
Links:
- added link left_tcp
- added link right_tcp
Joints:
- added joint left_tool0-tcp: type fixed, parent left_tool0, child left_tcp, origin xyz=0 0 0.24 rpy=0 0 0
- added joint right_tool0-tcp: type fixed, parent right_tool0, child right_tcp, origin xyz=0 0 0.24 rpy=0 0 0
